File: Adafruit Feather 328P.brd (EAGLE design)
At the start: 50.8 x 22.9 mm, 43 parts, among them IC1 CP2104, IC2 ATMEGA328P, Q3 DMG341, SW2 KMR2, U2 AP2112-3.3, U3 MCP73831T-2ACI/OT, X1 JSTPH, X4 20329, Y2 CSTCE16M0V53-R0 8MHZ

Commit message: fix https://github.com/adafruit/Adafruit-Feather-328P-PCB/issues/2
Parts:
- Y2: value CSTCE16M0V53-R0 8MHZ -> CSTNE8M00xx 8MHZ
Changed lines of the file:
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@@
 <?xml version="1.0" encoding="utf-8"?>
 <!DOCTYPE eagle SYSTEM "eagle.dtd">
-<eagle version="6.6.0">
+<eagle version="9.6.2">
 <drawing>
 <settings>
-<setting alwaysvectorfont="yes"/>
+<setting alwaysvectorfont="no"/>
+<setting keepoldvectorfont="yes"/>
 <setting verticaltext="up"/>
 </settings>
@@
 <layer number="59" name="tCarbon" color="7" fill="1" visible="no" active="no"/>
 <layer number="60" name="bCarbon" color="7" fill="1" visible="no" active="no"/>
-<layer number="90" name="Modules" color="7" fill="1" visible="no" active="yes"/>
+<layer number="90" name="Modules" color="7" fill="1" visible="no" active="no"/>
 <layer number="91" name="Nets" color="2" fill="1" visible="no" active="no"/>
 <layer number="92" name="Busses" color="1" fill="1" visible="no" active="no"/>
@@
 <param name="dpMaxLengthDifference" value="10mm"/>
 <param name="dpGapFactor" value="2.5"/>
-<param name="checkGrid" value="0"/>
 <param name="checkAngle" value="1"/>
 <param name="checkFont" value="1"/>
 <param name="checkRestrict" value="1"/>
+<param name="checkStop" value="0"/>
+<param name="checkValues" value="0"/>
+<param name="checkNames" value="1"/>
+<param name="checkWireStubs" value="1"/>
+<param name="checkPolygonWidth" value="0"/>
 <param name="useDiameter" value="13"/>
 <param name="maxErrors" value="50"/>
@@
 <pass name="Default">
 <param name="RoutingGrid" value="50mil"/>
+<param name="AutoGrid" value="1"/>
+<param name="Efforts" value="0"/>
+<param name="TopRouterVariant" value="1"/>
 <param name="tpViaShape" value="round"/>
 <param name="PrefDir.1" value="|"/>
@@
 <attribute name="VALUE" x="34.9885" y="9.779" size="0.8128" layer="27" font="vector" ratio="10" rot="R90"/>
 </element>
-<element name="Y2" library="SmartPrj" package="RESONATOR" value="CSTCE16M0V53-R0 8MHZ" x="33.2105" y="15.9766" smashed="yes" rot="R90">
+<element name="Y2" library="SmartPrj" package="RESONATOR" value="CSTNE8M00xx 8MHZ" x="33.2105" y="15.9766" smashed="yes" rot="R90">
 <attribute name="NAME" x="31.8605" y="14.5266" size="0.3556" layer="25" rot="R90"/>
 <attribute name="VALUE" x="32.0526" y="15.5205" size="0.8128" layer="27"/>
@@
 </element>
 <element name="IC2" library="microbuilder" package="MLF32-TH" value="ATMEGA328P" x="29.21" y="13.208" smashed="yes" rot="R180">
+<attribute name="MF" value="" x="29.21" y="13.208" size="1.778" layer="27" rot="R180" display="off"/>
+<attribute name="MPN" value="ATMEGA88PA-MU" x="29.21" y="13.208" size="1.778" layer="27" rot="R180" display="off"/>
+<attribute name="NAME" x="31.75" y="10.033" size="1.27" layer="25" rot="R180"/>
+<attribute name="OC_FARNELL" value="1715491" x="29.21" y="13.208" size="1.778" layer="27" rot="R180" display="off"/>
 <attribute name="OC_NEWARK" value="15R0272" x="29.21" y="13.208" size="1.778" layer="27" rot="R180" display="off"/>
-<attribute name="MPN" value="ATMEGA88PA-MU" x="29.21" y="13.208" size="1.778" layer="27" rot="R180" display="off"/>
-<attribute name="MF" value="" x="29.21" y="13.208" size="1.778" layer="27" rot="R180" display="off"/>
-<attribute name="OC_FARNELL" value="1715491" x="29.21" y="13.208" size="1.778" layer="27" rot="R180" display="off"/>
-<attribute name="NAME" x="31.75" y="10.033" size="1.27" layer="25" rot="R180"/>
 <attribute name="VALUE" x="31.877" y="12.954" size="0.8128" layer="27" rot="R180"/>
 </element>
@@
 <attribute name="VALUE" x="15.4305" y="5.207" size="0.8128" layer="27" font="vector" ratio="10" rot="R180"/>
 </element>
-<element name="U$44" library="microbuilder" package="ADAFRUIT_3.5MM" value="" x="3.429" y="9.779" rot="MR90"/>
+<element name="U$44" library="microbuilder" package="ADAFRUIT_3.5MM" value="" x="3.429" y="9.779" smashed="yes" rot="MR90"/>
 </elements>
 <signals>
@@
 <contactref element="X4" pad="SPRT@3"/>
 <contactref element="X4" pad="GND"/>
-<contactref element="X4" pad="SPRT@1"/>
-<contactref element="X4" pad="SPRT@2"/>
-<contactref element="X4" pad="BASE@1"/>
-<contactref element="X4" pad="SPRT@4"/>
-<contactref element="X4" pad="BASE@2"/>
-<contactref element="X4" pad="SPRT@3"/>
-<contactref element="X4" pad="GND"/>
-<contactref element="IC1" pad="2"/>
 <contactref element="C2" pad="2"/>
 <contactref element="IC1" pad="THERM"/>
@@
 <contactref element="IC2" pad="5"/>
 <contactref element="IC2" pad="21"/>
-<contactref element="IC2" pad="3"/>
-<contactref element="IC2" pad="5"/>
 <contactref element="IC2" pad="TH"/>
-<contactref element="IC2" pad="21"/>
 <via x="10.16" y="1.9685" extent="1-16" drill="0.3937"/>
 <via x="18.669" y="6.223" extent="1-16" drill="0.5"/>
@@
 <contactref element="IC1" pad="8"/>
 <contactref element="X4" pad="VBUS"/>
-<contactref element="X4" pad="VBUS"/>
-<contactref element="IC1" pad="8"/>
 <via x="15.4305" y="3.5052" extent="1-16" drill="0.5"/>
 <wire x1="15.0495" y1="10.668" x2="18.7325" y2="10.668" width="0.4064" layer="16"/>
@@
 <wire x1="11.684" y1="16.891" x2="12.7" y2="17.907" width="0.6096" layer="1"/>
 <wire x1="12.7" y1="17.907" x2="14.787" y2="17.907" width="0.6096" layer="1"/>
-<contactref element="U3" pad="3"/>
 <contactref element="U3" pad="3"/>
 <contactref element="Q3" pad="3"/>
@@
 </signal>
 </signals>
+<mfgpreviewcolors>
+<mfgpreviewcolor name="soldermaskcolor" color="0xC8008000"/>
+<mfgpreviewcolor name="silkscreencolor" color="0xFFFEFEFE"/>
+<mfgpreviewcolor name="backgroundcolor" color="0xFF282828"/>
+<mfgpreviewcolor name="coppercolor" color="0xFFFFBF00"/>
+<mfgpreviewcolor name="substratecolor" color="0xFF786E46"/>
+</mfgpreviewcolors>
 <errors>
 </errors>
